Commit message: updated urdf

File: src/robot_arm_control/robot_arm_control/urdf/robot_arm.urdf (robot description, URDF)
Before this commit: robot robot_arm, 7 links, 6 joints
Links:
- removed link Fixed_Gripper
- removed link Moving_Jaw
- removed link Shoulder_Rotation_Pitch
- added link Fixed_Jaw, mass 0.0929859131176897; collision mesh filename=package://robot_arm_control/meshes/Fixed_Jaw.STL; visual mesh filename=package://robot_arm_control/meshes/Fixed_Jaw.STL
- added link Moving Jaw, mass 0.0202443794940372; collision mesh filename=package://robot_arm_control/meshes/Moving_Jaw.STL; visual mesh filename=package://robot_arm_control/meshes/Moving_Jaw.STL
- added link Rotation_Pitch, mass 0.119226314127197; collision mesh filename=package://robot_arm_control/meshes/Rotation_Pitch.STL; visual mesh filename=package://robot_arm_control/meshes/Rotation_Pitch.STL
- link Base: mass 0.146962928243327 -> 0.193184127927598
- link Lower_Arm: mass 0.142523221917339 -> 0.147967774582291
- link Upper_Arm: mass 0.167601391353176 -> 0.162409284599177
- link Wrist_Pitch_Roll: mass 0.106401896179987 -> 0.066132067097723
Joints:
- removed joint Gripper
- removed joint Shoulder_Pitch
- removed joint Shoulder_Rotation
- added joint Jaw: type continuous, parent Fixed_Jaw, child Moving Jaw, origin xyz=-0.0202 -0.0244 0 rpy=3.1416 0 3.1416, axis 0 0 1
- added joint Pitch: type continuous, parent Rotation_Pitch, child Upper_Arm, origin xyz=0 0.1025 0.0306 rpy=0 0 0, axis 1 0 0
- added joint Rotation: type continuous, parent Base, child Rotation_Pitch, origin xyz=0 -0.0452 0.0165 rpy=1.5708 0 0, axis 0 1 0
- joint Elbow: axis 0 0 1 -> 1 0 0; origin xyz=-0.11238 0.0282 0 rpy=0 0 -2.2391 -> xyz=0 0.11257 0.028 rpy=0 0 0
- joint Wrist_Pitch: origin xyz=-0.1102 0.005375 0 rpy=0.90254 1.5708 0 -> xyz=0 0.0052 0.1349 rpy=0 0 0
- joint Wrist_Roll: axis 0 0 1 -> 0 1 0; child Fixed_Gripper -> Fixed_Jaw; origin xyz=0 0.002 -0.0545 rpy=3.1416 0 3.1416 -> xyz=0 -0.0601 0 rpy=0 0 0
