Commit message: rviz and urdf working

File: src/robot_arm_control/urdf/robot_arm.urdf (robot description, URDF)
Before this commit: robot robot_arm, 7 links, 6 joints
Joints:
- joint Rotation: axis 0 1 0 -> 0 -1 0
- joint Wrist_Pitch: origin xyz=0 0.0052 0.1349 rpy=0 0 0 -> xyz=0 0.0052 0.1349 rpy=-1.5708 0 0
- joint Wrist_Roll: origin xyz=0 -0.0601 0 rpy=0 0 0 -> xyz=0 -0.0601 0 rpy=0 1.5708 0
